File: Eagle files/tinyPixel - rev A.brd (EAGLE design)
At the start: 28.2 x 20.8 mm, 13 parts, among them IC1 ULN2003AD, U1 ATTINY85

Commit message: Updated Eagle files, BOM and Gerbers
Parts:
- moved R1 9.14 mm to (13.7, 9.65)
- moved JP3 5.08 mm to (11.7, 18.3), turned to 180 degrees
- moved R3 4.57 mm to (4.57, 9.65)
- moved R2 4.57 mm to (9.14, 9.65)
- moved JP5 0.25 mm to (16.0, 1.17)
- moved JP7 0.25 mm to (25.4, 10.4)
- moved JP6 0.20 mm to (11.4, 1.12), turned to 0 degrees
Connections:
- net B: now also JP3.3; no longer JP3.2
- net G: now also JP3.2; no longer JP3.3
Routing:
- net N$5: track 2.80 -> 11.6 mm, vias 0 -> 1
- net N$1: track 14.4 -> 8.43 mm
- net RESET: track 7.00 -> 4.62 mm, vias 2 -> 0
- net GND: track 1.86 -> 0.00 mm
- net G: track 3.28 -> 2.29 mm
- net B: track 2.29 -> 3.13 mm
- net N$3: track 9.26 -> 10.1 mm, vias 0 -> 1
Other:
- board text added: "REV A"
- board text removed: "bit.ly/YG8zBc"
