File: Eagle files/tinyPixel - rev A.sch (EAGLE design)
At the start: 12 parts, among them IC1 ULN2003AD, U1 ATTINY85

Commit message: Updated Eagle files, BOM and Gerbers
Connections:
- net B: now also JP3.3; no longer JP3.2
- net G: now also JP3.2; no longer JP3.3
Other:
- note added: "5V"
- note added: "GND"
- note added: "SCL"
- note added: "SDA"
- note removed: "RGB LED driver"
Changed lines of the file:
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@@
 <sheet>
 <plain>
-<text x="208.28" y="119.38" size="1.778" layer="97" font="vector">RGB LED driver</text>
+<text x="41.402" y="110.236" size="1.778" layer="97" rot="R180">5V</text>
+<text x="41.402" y="107.696" size="1.778" layer="97" rot="R180">GND</text>
+<text x="41.656" y="105.156" size="1.778" layer="97" rot="R180">SDA</text>
+<text x="41.656" y="102.616" size="1.778" layer="97" rot="R180">SCL</text>
 </plain>
 <instances>
@@
 </segment>
 </net>
-<net name="G" class="0">
-<segment>
-<pinref part="R2" gate="G$1" pin="2"/>
-<wire x1="205.74" y1="101.6" x2="205.74" y2="99.06" width="0.1524" layer="91"/>
-<pinref part="JP3" gate="G$1" pin="3"/>
-<wire x1="205.74" y1="99.06" x2="213.36" y2="99.06" width="0.1524" layer="91"/>
-<label x="210.82" y="99.06" size="1.778" layer="95"/>
-</segment>
-</net>
-<net name="B" class="0">
-<segment>
-<pinref part="JP3" gate="G$1" pin="2"/>
-<wire x1="213.36" y1="101.6" x2="208.28" y2="101.6" width="0.1524" layer="91"/>
-<wire x1="208.28" y1="101.6" x2="208.28" y2="91.44" width="0.1524" layer="91"/>
-<pinref part="R3" gate="G$1" pin="2"/>
-<wire x1="208.28" y1="91.44" x2="205.74" y2="91.44" width="0.1524" layer="91"/>
-<label x="210.82" y="101.6" size="1.778" layer="95"/>
-</segment>
-</net>
 <net name="RESET" class="0">
 <segment>
@@
 </segment>
 </net>
+<net name="B" class="0">
+<segment>
+<pinref part="R3" gate="G$1" pin="2"/>
+<wire x1="208.28" y1="91.44" x2="205.74" y2="91.44" width="0.1524" layer="91"/>
+<pinref part="JP3" gate="G$1" pin="3"/>
+<wire x1="213.36" y1="99.06" x2="208.28" y2="99.06" width="0.1524" layer="91"/>
+<wire x1="208.28" y1="99.06" x2="208.28" y2="91.44" width="0.1524" layer="91"/>
+<label x="210.82" y="99.06" size="1.778" layer="95"/>
+</segment>
+</net>
+<net name="G" class="0">
+<segment>
+<pinref part="R2" gate="G$1" pin="2"/>
+<pinref part="JP3" gate="G$1" pin="2"/>
+<wire x1="205.74" y1="101.6" x2="213.36" y2="101.6" width="0.1524" layer="91"/>
+<label x="210.82" y="101.6" size="1.778" layer="95"/>
+</segment>
+</net>
